File: twistedCharlieplex/twistedCharlieplex.kicad_pcb (KiCad board)
At the start: 6 copper layers, 38.9 x 38.9 mm, 145 parts, among them U2 STM32L412CBUxP

Commit message: Seconds LEDs are no more. This layout was actually trivial. I'm so upset. It's clean too.
Parts:
- removed D100, D101, D102, D103, D104, D105, D106, D107, D108, D109, D110, D111, D112, D113, D114, D115, D116, D117, D118, D119, D120, D61, D62, D63, D64, D65, D66, D67, D68, D69, D70, D71, D72, D73, D74, D75, D76, D77, D78, D79, D80, D81, D82, D83, D84, D85, D86, D87, D88, D89, D90, D91, D92, D93, D94, D95, D96, D97, D98, D99: LED_Small, LED_SMD:LED_0402_1005Metric
- D1, D10, D11, D12, D121, D122, D123, D124, D125, D126, D127, D128, D129, D13, D130, D131, D132, D133, D134, D135, D136, D137, D138, D139, D14, D140, D141, D142, D143, D144, D15, D16, D17, D18, D19, D2, D20, D21, D22, D23, D24, D25, D26, D27, D28, D29, D3, D30, D31, D32, D33, D34, D35, D36, D37, D38, D39, D4, D40, D41, D42, D43, D44, D45, D46, D47, D48, D49, D5, D50, D51, D52, D53, D54, D55, D56, D57, D58, D59, D6, D60, D7, D8, D9: footprint LED_SMD:LED_0402_1005Metric -> LED_SMD:LED_0603_1608Metric
- moved D126 4.14 mm to (-13.0, -3.48), turned to -105 degrees
- moved D132 4.14 mm to (-3.48, 13.0), turned to -15 degrees
- moved D138 4.14 mm to (13.0, 3.48), turned to 75 degrees
- moved D144 4.14 mm to (3.48, -13.0), turned to 165 degrees
- moved D122 4.14 mm to (-3.48, -13.0), turned to -165 degrees
- moved D128 4.14 mm to (-13.0, 3.48), turned to -75 degrees
- moved D134 4.14 mm to (3.48, 13.0), turned to 15 degrees
- moved D140 4.14 mm to (13.0, -3.48), turned to 105 degrees
- moved D121 4.14 mm to (0.00, -13.5), turned to 180 degrees
- moved D127 4.14 mm to (-13.5, 0.00), turned to -90 degrees
- moved D133 4.14 mm to (0.00, 13.5), turned to 0 degrees
- moved D139 4.14 mm to (13.5, 0.00), turned to 90 degrees
- moved D125 4.14 mm to (-11.7, -6.73), turned to -120 degrees
- moved D131 4.14 mm to (-6.73, 11.7), turned to -30 degrees
- moved D137 4.14 mm to (11.7, 6.73), turned to 60 degrees
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Routing:
- net /Charlie Displays/IO11: track 48.0 -> 0.00 mm, vias 16 -> 0
- net /Charlie Displays/IO12: track 47.2 -> 0.00 mm, vias 16 -> 0
- net /Charlie Displays/IO18: track 44.1 -> 0.00 mm, vias 18 -> 0
- net /Charlie Displays/IO16: track 36.6 -> 0.00 mm, vias 15 -> 0
- net /Charlie Displays/IO17: track 36.2 -> 0.00 mm, vias 16 -> 0
- net /Charlie Displays/IO7: track 38.4 -> 72.6 mm, vias 16 -> 14
- net /Charlie Displays/IO14: track 33.0 -> 0.00 mm, vias 15 -> 0
- net /Charlie Displays/IO25: track 10.1 -> 42.4 mm, vias 2 -> 5
- net /Charlie Displays/IO3: track 23.7 -> 55.0 mm
- net /Charlie Displays/IO5: track 28.5 -> 59.5 mm, vias 14 -> 12
- net /Charlie Displays/IO13: track 29.8 -> 0.00 mm, vias 13 -> 0
- net /Charlie Displays/IO15: track 29.6 -> 0.00 mm, vias 14 -> 0
- net /Charlie Displays/IO24: track 12.6 -> 41.9 mm, vias 1 -> 5
- net /Charlie Displays/IO23: track 7.65 -> 35.5 mm, vias 3 -> 5
- net /Charlie Displays/IO22: track 10.1 -> 34.5 mm, vias 2 -> 5
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Other:
- board size 38.9 x 38.9 mm -> 35.6 x 35.6 mm
