File: twistedCharlieplex/twistedCharlieplex.kicad_pcb (KiCad board)
At the start: 4 copper layers, 38.9 x 38.9 mm, 163 parts, among them Q1 Q_PMOS_GSD, U1 STM32L412CBUx, U2 LIS2DW12, U3 ESP32-C3, Y1 32.768k, Y2 40M

Commit message: Abandoning Attempt 3. This was AI
Parts:
- removed AE1: Antenna_Shield, Antenna_SMD:C209892
- removed C1, C3: 100n, Capacitor_SMD:C_0402_1005Metric
- removed C2: 10u, Capacitor_SMD:C_0402_1005Metric
- removed C4, C5: 4p3, Capacitor_SMD:C_0402_1005Metric
- removed C6, C7: 12p, Capacitor_SMD:C_0402_1005Metric
- removed Q1: Q_PMOS_GSD, Package_TO_SOT_SMD:SOT-523
- removed R1, R2, R3: 10k, Resistor_SMD:R_0402_1005Metric
- removed R4: 100k, Resistor_SMD:R_0402_1005Metric
- removed R5: 1M, Resistor_SMD:R_0402_1005Metric
- removed U1: STM32L412CBUx, Package_DFN_QFN:QFN-48-1EP_7x7mm_P0.5mm_EP5.6x5.6mm
- removed U2: LIS2DW12, Package_LGA:LGA-12_2x2mm_P0.5mm
- removed U3: ESP32-C3, Package_DFN_QFN:QFN-32-1EP_5x5mm_P0.5mm_EP3.7x3.7mm
- removed Y1: 32.768k, Crystal:Crystal_SMD_3215-2Pin_3.2x1.5mm
- removed Y2: 40M, SMD_Crystal:Crystal_SMD_1612_4P
Routing:
- net IO14: track 141.4 -> 15.9 mm, vias 17 -> 0
- net IO6: track 140.5 -> 16.0 mm, vias 16 -> 0
- net IO11: track 140.4 -> 17.7 mm, vias 15 -> 0
- net IO16: track 138.0 -> 16.0 mm, vias 16 -> 0
- net IO7: track 136.5 -> 16.0 mm, vias 15 -> 0
- net IO0: track 134.0 -> 13.4 mm, vias 15 -> 0
- net IO17: track 136.7 -> 16.4 mm, vias 15 -> 0
- net IO8: track 135.5 -> 16.4 mm, vias 17 -> 0
- net IO10: track 132.3 -> 13.4 mm, vias 15 -> 0
- net IO18: track 136.4 -> 18.1 mm, vias 16 -> 0
- net IO13: track 131.4 -> 13.4 mm, vias 13 -> 0
- net IO12: track 131.5 -> 13.9 mm, vias 17 -> 0
- net IO1: track 133.5 -> 17.7 mm, vias 15 -> 0
- net IO4: track 131.4 -> 16.0 mm, vias 16 -> 0
- net IO15: track 128.0 -> 13.5 mm, vias 13 -> 0
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Other:
- board text removed: "ring of fireeee"
